Commit message: Flatten track, keep camera tilt forward, rebuild images

File: ros2_ws/src/line_follower_robot/urdf/line_follower_bot.urdf.xacro (robot description, xacro)
@@ -28,4 +28,5 @@
   <link name="left_wheel_link">
     <visual>
+      <origin xyz="0 0 0" rpy="${pi/2} 0 0"/>
       <geometry>
         <cylinder radius="${wheel_radius}" length="${wheel_width}"/>
@@ -36,7 +37,16 @@
     </visual>
     <collision>
+      <origin xyz="0 0 0" rpy="${pi/2} 0 0"/>
       <geometry>
         <cylinder radius="${wheel_radius}" length="${wheel_width}"/>
       </geometry>
+      <surface>
+        <friction>
+          <ode>
+            <mu>1.0</mu>
+            <mu2>1.0</mu2>
+          </ode>
+        </friction>
+      </surface>
     </collision>
     <inertial>
@@ -47,4 +57,5 @@
   <link name="right_wheel_link">
     <visual>
+      <origin xyz="0 0 0" rpy="${pi/2} 0 0"/>
       <geometry>
         <cylinder radius="${wheel_radius}" length="${wheel_width}"/>
@@ -55,7 +66,16 @@
     </visual>
     <collision>
+      <origin xyz="0 0 0" rpy="${pi/2} 0 0"/>
       <geometry>
         <cylinder radius="${wheel_radius}" length="${wheel_width}"/>
       </geometry>
+      <surface>
+        <friction>
+          <ode>
+            <mu>1.0</mu>
+            <mu2>1.0</mu2>
+          </ode>
+        </friction>
+      </surface>
     </collision>
     <inertial>
@@ -88,17 +108,18 @@
     <parent link="base_link"/>
     <child link="left_wheel_link"/>
-    <origin xyz="0 ${wheel_sep/2.0} 0" rpy="0 ${pi/2} 0"/>
-    <axis xyz="0 0 1"/>
+    <origin xyz="0 ${wheel_sep/2.0} -0.017" rpy="0 0 0"/>
+    <axis xyz="0 1 0"/>
   </joint>
   <joint name="right_wheel_joint" type="continuous">
     <parent link="base_link"/>
     <child link="right_wheel_link"/>
-    <origin xyz="0 ${-wheel_sep/2.0} 0" rpy="0 ${pi/2} 0"/>
-    <axis xyz="0 0 1"/>
+    <origin xyz="0 ${-wheel_sep/2.0} -0.017" rpy="0 0 0"/>
+    <axis xyz="0 1 0"/>
   </joint>
   <joint name="camera_joint" type="fixed">
     <parent link="base_link"/>
     <child link="camera_link"/>
-    <origin xyz="0 0 0.15" rpy="${-0.6} 0 0"/>
+    <!-- Camera above robot, pitched ~45deg forward/down (negative pitch looks at ground ahead) -->
+    <origin xyz="0.08 0 0.22" rpy="0 ${0.785} 0"/>
   </joint>
   <!-- Transmissions -->
@@ -118,4 +139,7 @@
       <command_timeout>1.0</command_timeout>
       <odometry_frame>odom</odometry_frame>
+      <odometry_topic>odom</odometry_topic>
+      <publish_odom>true</publish_odom>
+      <publish_tf>true</publish_tf>
       <robot_base_frame>base_link</robot_base_frame>
     </plugin>
@@ -124,4 +148,5 @@
   <gazebo reference="camera_link">
     <sensor name="downward_camera" type="camera">
+      <!-- Sensor aligned with link; joint handles tilt -->
       <pose>0 0 0 0 0 0</pose>
       <visualize>true</visualize>

Commit message: Fix z-fighting floor, recenter camera, speed up line follower

File: ros2_ws/src/line_follower_robot/urdf/line_follower_bot.urdf.xacro (robot description, xacro)
@@ -121,5 +121,6 @@
     <child link="camera_link"/>
     <!-- Camera above robot, pitched ~45deg forward/down (negative pitch looks at ground ahead) -->
-    <origin xyz="0.08 0 0.22" rpy="0 ${0.785} 0"/>
+    <!-- Centered over base to avoid bias; keep 45deg pitch -->
+    <origin xyz="0 0 0.22" rpy="0 ${0.785} 0"/>
   </joint>
   <!-- Transmissions -->
